File: Amplifier_Circuit-V2/SensorArray_V2.kicad_pcb (KiCad board)
At the start: 4 copper layers, 84.1 x 60 mm, 102 parts, among them J1 UART_Connector, J2 Conn_02x05_Odd_Even, J3 I2C_Connector, J4 VCC_Connector, J5 SPI_Connector, J6 3V3_Connector, J7 Sensor_Array_Connector, J8 Sensor_Connector, J9 Amp_Sensor_out, SW1 SW_DIP_x01, U1 STM32F405RGTx, U10 CD74HC4067M, U2 AMS1117-3.3, U3 TLV71310PDBV, U4 INA326, U5 AD5272BRM, U6 CD74HC4067M, U7 AD5272BRM, U8 INA326, U9 MCP3562

Commit message: Sent to fabrication
Parts:
- removed the G*** at (97.0, 49.5)
- removed R18: 3k3, Resistor_SMD:R_0603_1608Metric
- added G***: LOGO, LogoSilkscreen:Logo_IMSAS4, F.Cu at (100.1, 58.2)
- added J10: SPI2_Connector, Connector_PinHeader_2.54mm:PinHeader_1x04_P2.54mm_Vertical, F.Cu at (60.0, 23.2)
- added J11: USB_B_Micro, Connector_USB:USB_Micro-B_Molex-105133-0001, F.Cu at (100.1, 36.1)
- added Q1: AO3401A, Package_TO_SOT_SMD:SOT-23, F.Cu at (90.6, 45.2)
- added R23: 100, Resistor_SMD:R_0402_1005Metric, F.Cu at (56.0, 43.5)
- added R24: 100, Resistor_SMD:R_0402_1005Metric, F.Cu at (56.1, 44.7)
- added R25: 100, Resistor_SMD:R_0402_1005Metric, F.Cu at (56.1, 45.8)
- added R26: 100, Resistor_SMD:R_0402_1005Metric, F.Cu at (56.1, 46.9)
- added U11: USBLC6-2SC6, Package_TO_SOT_SMD:SOT-23-6, F.Cu at (96.9, 43.6)
- J5: value SPI_Connector -> SPI1_Connector
- moved R_GND2 28.8 mm to (87.5, 76.4), turned to 180 degrees
- moved J6 13.6 mm to (86.4, 23.2)
- moved R2 13.5 mm to (79.0, 29.3), turned to 270 degrees
- moved J3 13.3 mm to (79.2, 23.2)
- moved F1 13.0 mm to (93.6, 48.4), turned to 180 degrees
- moved J9 12.7 mm to (71.9, 23.2)
- moved R1 12.2 mm to (80.7, 29.3), turned to 270 degrees
- moved C15 9.13 mm to (92.4, 39.1)
- moved D4 9.13 mm to (85.6, 30.4)
- moved R8 9.13 mm to (89.2, 30.4)
- moved U2 9.13 mm to (87.5, 36.5)
- moved C16 9.13 mm to (86.5, 42.0)
- moved FB1 9.13 mm to (90.8, 42.1)
- moved D3 8.03 mm to (90.3, 55.3)
- moved R7 8.03 mm to (90.3, 51.8)
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Connections:
- D2 pad 1: Net-(D2-Pad1) -> Vin
- D2 pad 2: VCC -> +5V
- F1 pad 1: Net-(D2-Pad1) -> VCC
- FB1 pad 2: Net-(F1-Pad2) -> Vin
- R7 pad 1: VCC -> Vin
- U1 pad 17: ADC_SPI1_CS -> ADC_SPI2_CS
- U1 pad 29: Net-(U1-Pad29) -> SPI2_SCK
- U1 pad 35: Net-(U1-Pad35) -> SPI2_MISO
- U1 pad 36: Net-(U1-Pad36) -> SPI2_MOSI
- U1 pad 44: Net-(U1-Pad44) -> USB_D-
- U1 pad 45: Net-(U1-Pad45) -> USB_D+
- U9 pad 13: ADC_SPI1_CS -> Net-(R26-Pad1)
- U9 pad 14: SPI1_SCK -> Net-(R25-Pad1)
- U9 pad 15: SPI1_MOSI -> Net-(R24-Pad1)
- U9 pad 16: SPI1_MISO -> Net-(R23-Pad1)
Routing:
- net SPI2_MOSI: track 0.00 -> 53.6 mm, vias 0 -> 3
- net SPI2_MISO: track 0.00 -> 47.5 mm, vias 0 -> 3
- net SPI2_SCK: track 0.00 -> 47.0 mm, vias 0 -> 3
- net ADC_SPI2_CS: track 0.00 -> 34.9 mm, vias 0 -> 2
- net AMP_OUT_B: track 54.8 -> 85.9 mm, vias 4 -> 3
- net USB_D-: track 0.00 -> 30.4 mm, vias 0 -> 2
- net USB_D+: track 0.00 -> 26.4 mm, vias 0 -> 2
- net +5V: track 0.00 -> 23.2 mm, vias 0 -> 2
- net GNDA: track 54.5 -> 76.9 mm
- net Vin: track 0.00 -> 15.3 mm
- net AMP_OUT_A: track 62.5 -> 74.9 mm
- net ADC_SPI1_CS: track 12.3 -> 0.00 mm
- net MUXA_S2: track 60.0 -> 70.0 mm
- net MUXA_S1: track 63.0 -> 73.0 mm
- net MUXA_S0: track 68.3 -> 78.3 mm
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Other:
- board text added: "CS_2"
- board text added: "Calibrate"
- board text added: "Hair Array Measurement Hair Sensor, Rev. 1 Minerva Vargas 2020"
- board text added: "MISO_2"
- board text added: "MOSI_2"
- board text added: "SCK_2"
- board text added: "SPI_1"
- board text added: "SPI_2"
- board text added: "Sensor Array"
- board text added: "Single Sensor"
- board text removed: "SPI"
