File: Amplifier_Circuit-V2/SensorArray_v2.sch (KiCad schematic (older format))
At the start: 38 parts, among them J1 UART_Connector, J2 Conn_02x05_Odd_Even, J3 I2C_Connector, J4 VCC_Connector, J5 SPI_Connector, J6 3V3_Connector, SW1 SW_DIP_x01, U1 STM32F405RGTx

Commit message: Sent to fabrication
Parts:
- added J10: SPI2_Connector, Connector_PinHeader_2.54mm:PinHeader_1x04_P2.54mm_Vertical, symbol SensorArray-rescue:Conn_01x04-Connector_Generic
- added J11: USB_B_Micro, Connector_USB:USB_Micro-B_Molex-105133-0001, symbol Connector:USB_B_Micro
- added U11: USBLC6-2SC6, Package_TO_SOT_SMD:SOT-23-6, symbol Power_Protection:USBLC6-2SC6
- J5: value SPI_Connector -> SPI1_Connector
Connections:
- net labels added: +5V, ADC_SPI2_CS, SPI2_MISO, SPI2_MOSI, SPI2_SCK, USB_CONN_D+, USB_CONN_D-, USB_D+, USB_D-
- net labels removed: ADC_SPI1_CS
- wire segments 122 -> 124
- no-connect marks 25 -> 22
Other:
- note added: "Crystal"
- note added: "I2C Pull resistors"
- note added: "USB with ESD protection"
- moved on the sheet: C1, C10, C11, C12, C13, C14, C2, C3, C4, C5, C6, C7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
